File: PCB/models-heart.kicad_pcb (KiCad board)
At the start: 4 copper layers, 21 x 32 mm, 59 parts, among them P1 USB_C_Plug, Q1 AO3401A, Q2 FS8205, Q3 UMH3N, Q4 AO3401A, Q5 AO3401A, Q6 BC857BS, Q7 BC857BS, Q8 AO3401A, Q9 UMH3N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

Commit message: Layout
Parts:
- added TP1: MOT A, TestPoint:TestPoint_Pad_D1.0mm, B.Cu at (71.0, 45.2)
- added TP10: +5V0, TestPoint:TestPoint_Pad_D1.0mm, B.Cu at (72.8, 51.5)
- added TP11: BTN, TestPoint:TestPoint_Pad_D1.0mm, B.Cu at (70.8, 49.2)
- added TP12: BTN, TestPoint:TestPoint_Pad_D1.0mm, B.Cu at (70.8, 51.5)
- added TP2: MOT B, TestPoint:TestPoint_Pad_D1.0mm, B.Cu at (71.0, 47.2)
- added TP3: BAT +, TestPoint:TestPoint_Pad_D1.0mm, B.Cu at (89.2, 49.2)
- added TP4: BAT -, TestPoint:TestPoint_Pad_D1.0mm, B.Cu at (87.2, 49.2)
- added TP5: BAT -, TestPoint:TestPoint_Pad_D1.0mm, B.Cu at (87.2, 51.5)
- added TP6: BAT +, TestPoint:TestPoint_Pad_D1.0mm, B.Cu at (89.2, 51.5)
- added TP7: GND, TestPoint:TestPoint_Pad_D1.0mm, B.Cu at (74.8, 49.2)
- added TP8: GND, TestPoint:TestPoint_Pad_D1.0mm, B.Cu at (74.8, 51.5)
- added TP9: +5V0, TestPoint:TestPoint_Pad_D1.0mm, B.Cu at (72.8, 49.2)
- moved Q4 16.0 mm to (87.8, 44.9)
- moved R13 16.0 mm to (90.2, 48.3)
- moved R14 16.0 mm to (90.2, 44.9)
- moved Q7 15.9 mm to (87.7, 48.4)
- moved Q5 15.9 mm to (71.7, 44.9)
- moved Q6 15.9 mm to (71.7, 48.4)
- moved R11 15.9 mm to (74.2, 48.3)
- moved R12 15.9 mm to (74.2, 44.9)
- moved R4 2.36 mm to (74.0, 53.6), turned to 90 degrees
- moved R7 1.81 mm to (71.6, 52.8)
- moved R9 1.81 mm to (71.6, 54.3)
- moved R3 1.69 mm to (82.4, 49.2)
Routing:
- net GND: track 0.45 -> 54.8 mm, vias 0 -> 40
- net +3V3: track 0.00 -> 25.4 mm, vias 0 -> 12
- net +PWR: track 0.00 -> 3.66 mm, vias 0 -> 4
- net BAT +: track 0.00 -> 2.99 mm, vias 0 -> 3
- net +5V0 USB: track 0.00 -> 2.83 mm, vias 0 -> 3
- net BAT -: track 0.00 -> 1.95 mm, vias 0 -> 2
- net +PWR (5V0 / 3V3): track 0.00 -> 1.49 mm, vias 0 -> 2

Commit message: minor fixes
Parts:
- moved Q1 15.2 mm to (87.2, 54.8), turned to 180 degrees
- moved R1 1.53 mm to (90.0, 54.9), turned to -90 degrees
- moved D2 1.50 mm to (88.8, 55.0)
- moved D1 0.76 mm to (88.8, 57.8)
- moved R2 0.64 mm to (89.2, 52.2)
- moved TP1 0.25 mm to (70.8, 45.2)
- moved TP2 0.25 mm to (70.8, 47.2)
Connections:
- net Net-(D3B-K) renamed BTN+
Routing:
- net +3V3: track 25.4 -> 64.2 mm
- net +PWR: track 3.66 -> 39.9 mm, vias 4 -> 6
- net +5V: track 0.00 -> 33.3 mm, vias 0 -> 7
- net BAT +: track 2.99 -> 34.3 mm, vias 3 -> 9
- net +PWR (5V0 / 3V3): track 1.49 -> 29.2 mm, vias 2 -> 6
- net +5V0 USB: track 2.83 -> 29.8 mm, vias 3 -> 9
- net BAT -: track 1.95 -> 25.4 mm, vias 2 -> 6
- net GND: track 54.8 -> 61.9 mm, vias 40 -> 43
- net BTN+: track 0.00 -> 6.99 mm, vias 0 -> 3
- net (no net): vias 30 -> 12
Other:
- board text added: "+"
- board text added: "+B-"
- board text added: "G"
- board text added: "M"
- board text added: "S"

Commit message: Release candidate
Parts:
- added TP13: OUT 5, TestPoint:TestPoint_Pad_D1.0mm, B.Cu at (77.0, 49.2)
- added TP14: OUT 4, TestPoint:TestPoint_Pad_D1.0mm, B.Cu at (79.0, 49.2)
- added TP15: OUT 3, TestPoint:TestPoint_Pad_D1.0mm, B.Cu at (81.0, 49.2)
- added TP16: OUT 2, TestPoint:TestPoint_Pad_D1.0mm, B.Cu at (83.0, 49.2)
- added TP17: OUT 1, TestPoint:TestPoint_Pad_D1.0mm, B.Cu at (85.0, 49.2)
- added TP18: GND, TestPoint:TestPoint_Pad_D1.0mm, B.Cu at (77.0, 46.5)
- added TP19: GND, TestPoint:TestPoint_Pad_D1.0mm, B.Cu at (85.0, 46.5)
- added TP20: GND, TestPoint:TestPoint_Pad_D1.0mm, B.Cu at (83.0, 46.5)
- added TP21: GND, TestPoint:TestPoint_Pad_D1.0mm, B.Cu at (81.0, 46.5)
- added TP22: GND, TestPoint:TestPoint_Pad_D1.0mm, B.Cu at (79.0, 46.5)
- added TP23: PWR, TestPoint:TestPoint_Pad_D1.0mm, B.Cu at (86.0, 47.8)
- added TP24: PWR, TestPoint:TestPoint_Pad_D1.0mm, B.Cu at (78.0, 47.8)
- added TP25: PWR, TestPoint:TestPoint_Pad_D1.0mm, B.Cu at (80.0, 47.8)
- added TP26: PWR, TestPoint:TestPoint_Pad_D1.0mm, B.Cu at (82.0, 47.8)
- added TP27: PWR, TestPoint:TestPoint_Pad_D1.0mm, B.Cu at (84.0, 47.8)
- moved R10 0.55 mm to (80.6, 46.8)
- moved C14 0.50 mm to (74.2, 29.5)
- moved C13 0.30 mm to (76.8, 29.5)
Routing:
- net LEFT_TURN_LIGHT_PIN: track 0.00 -> 33.0 mm, vias 0 -> 2
- net RIGHT_TURN_LIGHT_PIN: track 0.00 -> 29.3 mm, vias 0 -> 2
- net MOTOR_B: track 0.00 -> 23.1 mm, vias 0 -> 2
- net MOTOR_A: track 0.00 -> 23.0 mm, vias 0 -> 2
- net ESP GPIO 0: track 0.00 -> 22.4 mm, vias 0 -> 2
- net BTN+: track 6.99 -> 26.8 mm
- net GND: track 61.9 -> 79.4 mm, vias 43 -> 63
- net SERVO_PIN: track 0.00 -> 17.0 mm
- net HEAD_LIGHT_PIN: track 0.00 -> 15.9 mm, vias 0 -> 2
- net +PWR SENSE: track 0.00 -> 15.6 mm, vias 0 -> 1
- net +PWR: track 39.9 -> 55.4 mm
- net +3V3: track 64.2 -> 73.1 mm
- net +PWR HOLD: track 0.00 -> 8.74 mm
- net Net-(U1-TEMP): track 0.00 -> 7.93 mm
- net Net-(U5-EN): track 0.00 -> 6.98 mm, vias 0 -> 1
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Other:
- board text added: "B"
- board text removed: "+"
- board text removed: "+B-"
- board text removed: "G"
- board text removed: "S"

Commit message: Trace Almost Done
Parts:
- added TP28: +5V0, TestPoint:TestPoint_Pad_D1.0mm, F.Cu at (83.4, 51.3)
- added TP29: +5V0, TestPoint:TestPoint_Pad_D1.0mm, F.Cu at (68.3, 58.0)
- added TP30: RX, TestPoint:TestPoint_Pad_D1.0mm, F.Cu at (67.9, 30.0)
- added TP31: TX, TestPoint:TestPoint_Pad_D1.0mm, F.Cu at (70.7, 28.0)
- added TP32: RX, TestPoint:TestPoint_Pad_D1.0mm, F.Cu at (70.7, 30.0)
- added TP33: TX, TestPoint:TestPoint_Pad_D1.0mm, F.Cu at (67.9, 28.0)
- added TP34: RST, TestPoint:TestPoint_Pad_D1.0mm, F.Cu at (70.7, 32.0)
- added TP35: RST, TestPoint:TestPoint_Pad_D1.0mm, F.Cu at (67.9, 32.0)
- added TP36: IO 0, TestPoint:TestPoint_Pad_D1.0mm, F.Cu at (70.8, 34.0)
- added TP37: IO 0, TestPoint:TestPoint_Pad_D1.0mm, F.Cu at (67.9, 34.0)
- added TP38: D-, TestPoint:TestPoint_Pad_D1.0mm, F.Cu at (64.3, 58.0)
- added TP39: D-, TestPoint:TestPoint_Pad_D1.0mm, F.Cu at (79.4, 51.3)
- added TP40: D+, TestPoint:TestPoint_Pad_D1.0mm, F.Cu at (66.3, 58.0)
- added TP41: D+, TestPoint:TestPoint_Pad_D1.0mm, F.Cu at (81.4, 51.3)
- added TP42: GND, TestPoint:TestPoint_Pad_D1.0mm, F.Cu at (77.4, 51.3)
- added TP43: GND, TestPoint:TestPoint_Pad_D1.0mm, F.Cu at (62.3, 58.0)
- moved C3 7.05 mm to (63.7, 49.1), turned to 0 degrees
- moved C4 4.38 mm to (63.9, 47.0)
- moved Q3 4.37 mm to (64.0, 33.6)
- moved U3 4.27 mm to (65.0, 40.4)
- moved R5 3.01 mm to (64.1, 29.8)
- moved R6 3.01 mm to (64.1, 28.3)
- moved C8 0.19 mm to (71.9, 35.7)
- moved R15 0.14 mm to (71.8, 37.2)
- moved R19 0.14 mm to (71.8, 38.7)
- moved R24 0.14 mm to (71.8, 40.7)
Routing:
- net /USB D+: track 0.00 -> 48.8 mm, vias 0 -> 4
- net /USB D-: track 0.00 -> 48.8 mm, vias 0 -> 4
- net ESP RST: track 3.92 -> 31.8 mm, vias 1 -> 3
- net +5V: track 33.3 -> 59.1 mm, vias 7 -> 12
- net MOT A: track 0.00 -> 19.8 mm, vias 0 -> 5
- net Net-(U3-TXD): track 0.00 -> 19.4 mm, vias 0 -> 2
- net Net-(U3-RXD): track 0.00 -> 19.4 mm, vias 0 -> 2
- net RTS: track 0.00 -> 14.5 mm, vias 0 -> 2
- net BTN+: track 26.8 -> 40.5 mm, vias 3 -> 4
- net DTR: track 0.00 -> 11.8 mm
- net ESP GPIO 0: track 22.4 -> 33.9 mm, vias 2 -> 7
- net ESP RxD: track 0.00 -> 9.18 mm, vias 0 -> 2
- net MOT B: track 0.65 -> 9.35 mm, vias 0 -> 5
- net ESP TxD: track 0.00 -> 8.55 mm, vias 0 -> 3
- net GND: track 79.4 -> 83.7 mm, vias 63 -> 69
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Other:
- board size 21 x 32 mm -> 29.9 x 32 mm

Commit message: PCB Done
Parts:
- C14: footprint Capacitor_SMD:C_1206_3216Metric -> Capacitor_SMD:C_0805_2012Metric
- moved R22 2.00 mm to (73.2, 40.7), turned to 0 degrees
- moved R24 1.62 mm to (71.5, 42.3)
- moved C14 0.47 mm to (74.2, 29.1)
- moved R13 0.25 mm to (90.0, 48.3)
- moved C13 0.24 mm to (76.6, 29.7)
- moved C9 0.21 mm to (89.3, 28.0)
- moved R12 0.12 mm to (74.3, 45.0)
- moved R17 0.10 mm to (89.3, 29.4)
- moved R3 0.10 mm to (82.4, 49.3)
- moved TP34 0.10 mm to (70.8, 32.0)
Routing:
- net GND: track 83.7 -> 97.6 mm, vias 69 -> 88
- net MOT B: track 9.35 -> 19.3 mm
- net +PWR: track 55.4 -> 61.7 mm, vias 6 -> 10
- net +3V3: track 73.7 -> 67.9 mm, vias 12 -> 13
- net +PWR (5V0 / 3V3): track 34.4 -> 39.4 mm
- net ESP ADC: track 1.50 -> 5.02 mm, vias 0 -> 1
- net +PWR HOLD: track 10.7 -> 14.2 mm, vias 0 -> 1
- net BAT +: track 36.2 -> 39.5 mm
- net ESP GPIO 0: track 33.9 -> 37.1 mm
- net MOT A: track 19.8 -> 22.2 mm
- net BAT -: track 25.8 -> 23.5 mm, vias 6 -> 5
- net HEAD_LIGHT_PIN: track 14.9 -> 17.0 mm, vias 2 -> 3
- net Net-(U6-VINT): track 2.31 -> 3.94 mm
- net LEFT_TURN_LIGHT_PIN: track 32.8 -> 34.1 mm
- net BTN+: track 40.5 -> 39.2 mm, vias 4 -> 3
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- added copper zone on F.Cu, net +3V3
- added copper zone on In2.Cu, net +3V3
- added copper zone on In2.Cu, net +5V
- added copper zone on In2.Cu, net +5V0 USB
- added copper zone on B.Cu, net +PWR
- added copper zone on F.Cu, net +PWR
- added copper zone on In2.Cu, net +PWR
- added copper zone on In2.Cu, net +PWR (5V0 / 3V3)
- added copper zone on In2.Cu, net BAT +
- added copper zone on In2.Cu, net BAT -
- added copper zone on B.Cu, net GND
- added copper zone on F.Cu, net GND
- added copper zone on In2.Cu, net GND
- added copper zone on B.Cu, net MOT A
- added copper zone on F.Cu, net MOT A
- added copper zone on In2.Cu, net MOT A
- added copper zone on B.Cu, net MOT B
- added copper zone on F.Cu, net MOT B
- added copper zone on In2.Cu, net MOT B

Commit message: Production
Other:
- board text added: "Open Source Heart of Model"
- board text added: "REV 1"
- board text removed: "B"
