File: PCB/models-heart.kicad_pcb (KiCad board)
At the start: 4 copper layers, 29.9 x 32 mm, 102 parts, among them P1 USB_C_Plug, Q1 AO3401A, Q2 FS8205, Q3 UMH3N, Q4 AO3401A, Q5 AO3401A, Q6 BC857BS, Q7 BC857BS, Q8 AO3401A, Q9 UMH3N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

Commit message: Fabrication
Parts:
- moved R3 1.74 mm to (84.2, 49.1), turned to 180 degrees
Connections:
- D3 pad 1: unconnected-(D3A-A-Pad1) -> Net-(D3A-A)
- D3 pad 6: unconnected-(D3A-K-Pad6) -> BTN+
- Q8 pad 1: BTN+ -> Net-(D3A-A)
- Q9 pad 6: BTN+ -> Net-(D3A-A)
- R23 pad 2: BTN+ -> Net-(D3A-A)
Routing:
- net Net-(D3A-A): track 0.00 -> 11.9 mm
- net BTN+: track 39.2 -> 31.6 mm
- net LEFT_TURN_LIGHT_PIN: track 34.1 -> 31.1 mm
- net BAT -: track 23.5 -> 24.7 mm, vias 5 -> 7
- net +5V0 USB: track 31.1 -> 31.8 mm
- net +PWR SENSE: track 15.6 -> 16.2 mm
- net Net-(Q4-G): track 5.28 -> 5.79 mm
- net BAT +: track 39.5 -> 39.6 mm, vias 9 -> 12
- net GND: vias 88 -> 91
- added copper zone on B.Cu, net BAT +
- added copper zone on F.Cu, net BAT +

Commit message: Production Complete
Routing:
- net +5V0 USB: track 31.8 -> 42.0 mm, vias 8 -> 17
- net +PWR (5V0 / 3V3): track 39.6 -> 46.4 mm, vias 6 -> 11
- net +5V: track 59.7 -> 63.7 mm, vias 12 -> 16
- net +PWR: track 61.7 -> 64.0 mm, vias 10 -> 12
- added copper zone on B.Cu, net +5V
- added copper zone on F.Cu, net +5V
- added copper zone on B.Cu, net +5V0 USB
- added copper zone on F.Cu, net +5V0 USB
- added copper zone on B.Cu, net BAT -
- added copper zone on F.Cu, net BAT -
Other:
- board text added: "Віталіку Від Іруськи"
- board text added: "Дякую Ірусці за підтримку під час роботи над проєктом"

Commit message: Part 5
Other:
- board text added: "Дякую Ірусьці за підтримку під час роботи над проєктом"
- board text removed: "Дякую Ірусці за підтримку під час роботи над проєктом"
Changed lines of the file:
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@@
     (effects (font (size 1.1 1.1) (thickness 0.15)) (justify left bottom mirror))
   )
-  (gr_text "Дякую Ірусці\nза підтримку\nпід час роботи \nнад проєктом" (at 63.2 56.5 270) (layer "B.SilkS")
+  (gr_text "Дякую Ірусьці\nза підтримку\nпід час роботи \nнад проєктом" (at 63.2 56.7 270) (layer "B.SilkS")
     (effects (font (size 0.7 0.6) (thickness 0.1)) (justify left bottom mirror))
   )
