File: PCB/models-heart.kicad_pcb (KiCad board)
At the start: 4 copper layers, 29.9 x 32 mm, 106 parts, among them P1 USB_C_Plug, Q1 AO3401A, Q2 FS8205, Q3 UMH3N, Q4 AO3401A, Q5 AO3401A, Q6 BC857BS, Q7 BC857BS, Q8 AO3401A, Q9 UMH3N, SW1 SW_Push, U1 TP4056, U2 DW01, U3 CH340C, U4 AMS1117-3.3, U5 ESP-12E, U6 DRV8833PWP

Commit message: actionns test
Connections:
- P1 pad B6: (no net) -> /USB D+
- P1 pad B7: (no net) -> /USB D-
Routing:
- net /USB D-: track 49.2 -> 52.5 mm
- net /USB D+: track 49.0 -> 51.8 mm

Commit message: REV2
Parts:
- removed P1: USB_C_Plug, Connector_USB:USB_C_Receptacle_GCT_USB4105-xx-A_16P_TopMnt_Horizontal
- removed TP12: BTN, TestPoint:TestPoint_Pad_D1.0mm
- removed TP28, TP29, TP9: +5V0, TestPoint:TestPoint_Pad_D1.0mm
- removed TP30, TP32: RX, TestPoint:TestPoint_Pad_D1.0mm
- removed TP31, TP33: TX, TestPoint:TestPoint_Pad_D1.0mm
- removed TP34, TP35: RST, TestPoint:TestPoint_Pad_D1.0mm
- removed TP36, TP37: IO 0, TestPoint:TestPoint_Pad_D1.0mm
- removed TP38, TP39: D-, TestPoint:TestPoint_Pad_D1.0mm
- removed TP40, TP41: D+, TestPoint:TestPoint_Pad_D1.0mm
- removed TP42, TP43, TP7: GND, TestPoint:TestPoint_Pad_D1.0mm
- added C16: 0.1uF, Capacitor_SMD:C_0603_1608Metric, F.Cu at (115.5, 58.3)
- added C17: 0.1uF, Capacitor_SMD:C_0603_1608Metric, F.Cu at (117.0, 54.2)
- added J1: USB_C_Receptacle, Connector_USB:USB_C_Receptacle_GCT_USB4115-03-C, F.Cu at (121.0, 67.1)
- added R29: 15k, Resistor_SMD:R_0603_1608Metric, F.Cu at (118.5, 54.2)
- added R30: 100k, Resistor_SMD:R_0603_1608Metric, F.Cu at (115.5, 54.2)
- added U7: TPS3808DBV, Package_TO_SOT_SMD:SOT-23-6, F.Cu at (118.0, 57.8)
- C1, C15, C3, C4, Q3, R8, U1, U3: moved to B.Cu
- C2: value 10uF -> 0.1uF; footprint Capacitor_SMD:C_1206_3216Metric -> Capacitor_SMD:C_0603_1608Metric; moved to B.Cu
- D1, D2, SW1: moved to F.Cu
- R16: value 10k -> 100k
- TP5: value BAT - -> GND
- TP6: value BAT + -> NTC
- moved C3 65.1 mm to (128.2, 57.8), turned to -90 degrees
- moved TP11 63.7 mm to (132.0, 67.0)
- moved C4 63.3 mm to (126.7, 55.0), turned to 180 degrees
- moved U3 60.4 mm to (122.2, 60.0), turned to 90 degrees
- moved TP8 59.8 mm to (132.0, 69.0)
- moved SW1 58.6 mm to (130.2, 68.3), turned to 0 degrees
- moved R26 57.5 mm to (128.2, 68.4), turned to -90 degrees
- moved Q3 57.2 mm to (114.8, 60.0), turned to -90 degrees
- moved C15 55.8 mm to (121.0, 64.5), turned to 180 degrees
- moved R27 55.7 mm to (126.7, 68.4), turned to -90 degrees
- moved Q2 55.3 mm to (130.5, 62.1), turned to 180 degrees
- moved TP24 54.1 mm to (132.0, 44.5), turned to -90 degrees
- moved R10 53.6 mm to (131.1, 64.6), turned to 0 degrees
- moved TP25 52.3 mm to (132.0, 42.5), turned to -90 degrees
- moved TP10 52.2 mm to (122.0, 69.0)
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Connections:
- C2 pad 1: GND -> BAT +
- C2 pad 2: BAT + -> GND
- R18 pad 1: +3V3 -> Net-(U5-EN)
- R18 pad 2: Net-(U5-EN) -> +3V3
- TP5 pad 1: BAT - -> GND
- TP6 pad 1: BAT + -> Net-(U1-TEMP)
Routing:
- net GND: track 98.1 -> 0.00 mm, vias 92 -> 0
- net +3V3: track 69.8 -> 0.00 mm, vias 14 -> 0
- net +PWR: track 64.0 -> 0.00 mm, vias 12 -> 0
- net +5V: track 63.8 -> 0.00 mm, vias 16 -> 0
- net /USB D-: track 52.5 -> 0.00 mm, vias 4 -> 0
- net /USB D+: track 51.8 -> 0.00 mm, vias 4 -> 0
- net +PWR (5V0 / 3V3): track 46.3 -> 0.00 mm, vias 11 -> 0
- net +5V0 USB: track 42.1 -> 0.00 mm, vias 17 -> 0
- net BAT +: track 40.0 -> 0.00 mm, vias 12 -> 0
- net ESP GPIO 0: track 37.1 -> 0.00 mm, vias 7 -> 0
- net ESP RST: track 32.7 -> 0.00 mm, vias 3 -> 0
- net BTN+: track 31.6 -> 0.00 mm, vias 3 -> 0
- net LEFT_TURN_LIGHT_PIN: track 31.1 -> 0.00 mm, vias 2 -> 0
- net RIGHT_TURN_LIGHT_PIN: track 27.3 -> 0.00 mm, vias 2 -> 0
- net BAT -: track 24.7 -> 0.00 mm, vias 7 -> 0
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- removed copper zone on F.Cu, net +3V3
- removed copper zone on In2.Cu, net +3V3
- removed copper zone on B.Cu, net +5V
- removed copper zone on F.Cu, net +5V
- removed copper zone on In2.Cu, net +5V
- removed copper zone on B.Cu, net +5V0 USB
- removed copper zone on F.Cu, net +5V0 USB
- removed copper zone on In2.Cu, net +5V0 USB
- removed copper zone on B.Cu, net +PWR
- removed copper zone on F.Cu, net +PWR
- removed copper zone on In2.Cu, net +PWR
- removed copper zone on In2.Cu, net +PWR (5V0 / 3V3)
- removed copper zone on B.Cu, net BAT +
- removed copper zone on F.Cu, net BAT +
- removed copper zone on In2.Cu, net BAT +
- removed copper zone on B.Cu, net BAT -
- removed copper zone on F.Cu, net BAT -
- removed copper zone on In2.Cu, net BAT -
- removed copper zone on B.Cu, net GND
- removed copper zone on F.Cu, net GND
- removed copper zone on In1.Cu, net GND
- removed copper zone on In2.Cu, net GND
- removed copper zone on B.Cu, net MOT A
- removed copper zone on F.Cu, net MOT A
- removed copper zone on In2.Cu, net MOT A
- removed copper zone on B.Cu, net MOT B
- removed copper zone on F.Cu, net MOT B
- removed copper zone on In2.Cu, net MOT B
Other:
- board size 29.9 x 32 mm -> 24 x 35 mm
- board text added: "1"
- board text added: "2"
- board text added: "3"
- board text added: "4"
- board text added: "5"
- board text added: "REV ${REVISION}"
- board text removed: "REV 1"
- board text removed: "Віталіку Від Іруськи"

Commit message: placement
Parts:
- removed TP26, TP27: PWR, TestPoint:TestPoint_Pad_D1.0mm
- added H1: MountingHole, MountingHole:MountingHole_2.2mm_M2, F.Cu at (131.2, 32.4)
- added H2: MountingHole, MountingHole:MountingHole_2.2mm_M2, F.Cu at (110.8, 32.5)
- added H3: MountingHole_Pad, MountingHole:MountingHole_2.2mm_M2_Pad_Via, F.Cu at (111.5, 67.5)
- added H4: MountingHole_Pad, MountingHole:MountingHole_2.2mm_M2_Pad_Via, F.Cu at (130.5, 67.5)
- added TP12: GND, TestPoint:TestPoint_Pad_D1.0mm, B.Cu at (132.0, 50.0)
- added TP28: GND, TestPoint:TestPoint_Pad_D1.0mm, B.Cu at (132.0, 38.0)
- added TP29: GND, TestPoint:TestPoint_Pad_D1.0mm, B.Cu at (132.0, 42.0)
- added TP7: GND, TestPoint:TestPoint_Pad_D1.0mm, B.Cu at (132.0, 54.0)
- added TP9: PWR, TestPoint:TestPoint_Pad_D1.0mm, B.Cu at (132.0, 52.0)
- C11, C12, C15, C16, C17, C3, C7, C8, C9: value 0.1uF -> 100n; footprint Capacitor_SMD:C_0603_1608Metric -> Capacitor_SMD:C_0402_1005Metric
- C2: value 0.1uF -> 10uF; footprint Capacitor_SMD:C_0603_1608Metric -> Capacitor_SMD:C_1206_3216Metric
- R1, R10, R11, R12, R13, R14, R15, R16, R17, R18, R19, R2, R20, R21, R22, R23, R24, R25, R28, R29, R3, R30, R4, R5, R6, R7, R8: footprint Resistor_SMD:R_0603_1608Metric -> Resistor_SMD:R_0402_1005Metric
- R26, R27: footprint Resistor_SMD:R_0603_1608Metric -> Resistor_SMD:R_0402_1005Metric; moved to F.Cu
- SW1: footprint Button_Switch_SMD:SW_SPST_EVQP7C -> Button_Switch_SMD:SW_Push_SPST_NO_Alps_SKRK
- moved TP17 23.2 mm to (132.0, 44.0)
- moved TP19 23.2 mm to (132.0, 46.0)
- moved SW1 11.7 mm to (121.0, 61.1), turned to -90 degrees
- moved TP8 6.80 mm to (125.2, 69.0)
- moved D2 5.30 mm to (112.2, 61.5), turned to 0 degrees
- moved R21 5.24 mm to (131.0, 38.2)
- moved U1 5.20 mm to (112.0, 61.0)
- moved TP11 5.20 mm to (127.2, 69.0)
- moved R2 5.11 mm to (114.8, 61.7), turned to 180 degrees
- moved R8 5.10 mm to (111.9, 56.6)
- moved R18 4.70 mm to (131.0, 41.8), turned to 0 degrees
- moved C15 4.61 mm to (125.2, 62.6), turned to 0 degrees
- moved R24 4.51 mm to (110.9, 47.1)
- moved TP1 4.50 mm to (110.0, 52.0)
- moved TP13 4.50 mm to (110.0, 48.0)
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Connections:
- C2 pad 1: BAT + -> GND
- C2 pad 2: GND -> BAT +
Routing:
- net GND: track 0.00 -> 0.65 mm, vias 0 -> 1
Other:
- board size 24 x 35 mm -> 24 x 39.4 mm
- board text added: "ON/OFF"
- board text added: "x"
- board text removed: "Дякую Ірусьці за підтримку під час роботи над проєктом"
