File: PCB/models-heart.kicad_sch (KiCad schematic)
At the start: 60 parts, among them P1 USB_C_Plug, Q1 AO3401A, Q2 FS8205, Q3 UMH3N, Q4 AO3401A, Q5 AO3401A, Q6 BC857BS, Q7 BC857BS, Q8 AO3401A, Q9 UMH3N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

Commit message: Layout
Parts:
- added TP1: MOT A, TestPoint:TestPoint_Pad_D1.0mm, symbol Connector:TestPoint_Small
- added TP10, TP9: +5V0, TestPoint:TestPoint_Pad_D1.0mm, symbol Connector:TestPoint_Small
- added TP11, TP12: BTN, TestPoint:TestPoint_Pad_D1.0mm, symbol Connector:TestPoint_Small
- added TP2: MOT B, TestPoint:TestPoint_Pad_D1.0mm, symbol Connector:TestPoint_Small
- added TP3, TP6: BAT +, TestPoint:TestPoint_Pad_D1.0mm, symbol Connector:TestPoint_Small
- added TP4, TP5: BAT -, TestPoint:TestPoint_Pad_D1.0mm, symbol Connector:TestPoint_Small
- added TP7, TP8: GND, TestPoint:TestPoint_Pad_D1.0mm, symbol Connector:TestPoint_Small
Connections:
- net +5V0 USB: now also TP10.1, TP9.1
- net BAT +: now also TP3.1, TP6.1
- net BAT -: now also TP4.1, TP5.1
- net GND: now also TP7.1, TP8.1
- net MOT A: now also TP1.1
- net MOT B: now also TP2.1
- net at D3.5 (K), Q8.1 (G), Q9.6 (C1)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: now also TP11.1, TP12.1
Other:
- moved on the sheet: SW1

Commit message: Schematic
Other:
- note added: "Model's Heart"
- note removed: "Model Heart"
- company: (none) -> kushlavr@gmail.com
- title: Model Heart -> Model's Heart
Changed lines of the file:
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@@
   (paper "A3")
   (title_block
-    (title "Model Heart")
+    (title "Model's Heart")
     (rev "1")
+    (company "kushlavr@gmail.com")
+    (comment 1 "https://github.com/KushlaVR/models-heart")
   )
   (junction (at 200.66 78.74) (diameter 0) (color 0 0 0 0)
@@
     (effects (font (size 1.27 1.27)) (justify left bottom))
   )
-  (text "Model Heart" (at 312.42 265.43 0)
-    (effects (font (size 8 8)) (justify left bottom))
+  (text "Model's Heart" (at 299.72 262.89 0)
+    (effects (font (size 7 7)) (justify left bottom))
   )
   (text "0" (at 76.2 157.48 0)

Commit message: minor fixes
Connections:
- net BTN+: now reaches D3.5 (K), Q8.1 (G), Q9.6 (C1), R23.2, SW1.1, TP11.1, TP12.1
Changed lines of the file:
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@@
   (junction (at 345.44 50.8) (diameter 0) (color 0 0 0 0)
+  )
+  (junction (at 358.14 177.8) (diameter 0) (color 0 0 0 0)
   )
   (junction (at 199.39 148.59) (diameter 0) (color 0 0 0 0)
@@
     (stroke (width 0) (type default))
   )
+  (wire (pts (xy 358.14 177.8) (xy 365.76 177.8))
+    (stroke (width 0) (type default))
+  )
   (wire (pts (xy 339.09 196.85) (xy 350.52 196.85))
     (stroke (width 0) (type default))
@@
     (stroke (width 0) (type default))
   )
-  (wire (pts (xy 355.6 177.8) (xy 365.76 177.8))
+  (wire (pts (xy 355.6 177.8) (xy 358.14 177.8))
     (stroke (width 0) (type default))
   )
@@
     (stroke (width 0) (type default))
   )
+  (wire (pts (xy 358.14 180.34) (xy 358.14 177.8))
+    (stroke (width 0) (type default))
+  )
   (wire (pts (xy 152.4 219.71) (xy 161.29 219.71))
     (stroke (width 0) (type default))
@@
   )
   (wire (pts (xy 314.96 64.77) (xy 314.96 62.23))
+    (stroke (width 0) (type default))
+  )
+  (wire (pts (xy 360.68 180.34) (xy 358.14 180.34))
     (stroke (width 0) (type default))
   )
@@
       (effects (font (size 1.27 1.27)) (justify left) hide)
     )
+  )
+  (global_label "BTN+" (shape input) (at 360.68 180.34 0) (fields_autoplaced)
+    (effects (font (size 1.27 1.27)) (justify left))
+    (property "Intersheetrefs" "${INTERSHEET_REFS}" (at 368.7263 180.34 0)
+      (effects (font (size 1.27 1.27)) (justify left) hide)
+    )

Commit message: Release candidate
Parts:
- added TP13: OUT 5, TestPoint:TestPoint_Pad_D1.0mm, symbol Connector:TestPoint_Small
- added TP14: OUT 4, TestPoint:TestPoint_Pad_D1.0mm, symbol Connector:TestPoint_Small
- added TP15: OUT 3, TestPoint:TestPoint_Pad_D1.0mm, symbol Connector:TestPoint_Small
- added TP16: OUT 2, TestPoint:TestPoint_Pad_D1.0mm, symbol Connector:TestPoint_Small
- added TP17: OUT 1, TestPoint:TestPoint_Pad_D1.0mm, symbol Connector:TestPoint_Small
- added TP18, TP19, TP20, TP21, TP22: GND, TestPoint:TestPoint_Pad_D1.0mm, symbol Connector:TestPoint_Small
- added TP23, TP24, TP25, TP26, TP27: PWR, TestPoint:TestPoint_Pad_D1.0mm, symbol Connector:TestPoint_Small
Connections:
- net +PWR: now also TP23.1, TP24.1, TP25.1, TP26.1, TP27.1
- net ESP GPIO 0: now also TP13.1
- net GND: now also TP18.1, TP19.1, TP20.1, TP21.1, TP22.1
- net HEAD_LIGHT_PIN: now also TP14.1
- net LEFT_TURN_LIGHT_PIN: now also TP16.1
- net RIGHT_TURN_LIGHT_PIN: now also TP15.1
- net SERVO_PIN: now also TP17.1
Other:
- note added: "GPIO Solder Points"

Commit message: Trace Almost Done
Parts:
- added TP28, TP29: +5V0, TestPoint:TestPoint_Pad_D1.0mm, symbol Connector:TestPoint_Small
- added TP30, TP32: RX, TestPoint:TestPoint_Pad_D1.0mm, symbol Connector:TestPoint_Small
- added TP31, TP33: TX, TestPoint:TestPoint_Pad_D1.0mm, symbol Connector:TestPoint_Small
- added TP34, TP35: RST, TestPoint:TestPoint_Pad_D1.0mm, symbol Connector:TestPoint_Small
- added TP36, TP37: IO 0, TestPoint:TestPoint_Pad_D1.0mm, symbol Connector:TestPoint_Small
- added TP38, TP39: D-, TestPoint:TestPoint_Pad_D1.0mm, symbol Connector:TestPoint_Small
- added TP40, TP41: D+, TestPoint:TestPoint_Pad_D1.0mm, symbol Connector:TestPoint_Small
- added TP42, TP43: GND, TestPoint:TestPoint_Pad_D1.0mm, symbol Connector:TestPoint_Small
Connections:
- net +5V: now also TP28.1, TP29.1
- net ESP GPIO 0: now also TP36.1, TP37.1
- net ESP RST: now also TP34.1, TP35.1
- net ESP RxD: now also TP30.1, TP32.1
- net ESP TxD: now also TP31.1, TP33.1
- net GND: now also TP42.1, TP43.1
- net USB D+: now also TP40.1, TP41.1
- net USB D-: now also TP38.1, TP39.1
Other:
- moved on the sheet: P1, Q1, TP10, TP7, TP8, TP9

Commit message: PCB Done
Parts:
- C14: footprint Capacitor_SMD:C_1206_3216Metric -> Capacitor_SMD:C_0805_2012Metric
Changed lines of the file:
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@@
       (effects (font (size 1.27 1.27)) (justify left))
     )
-    (property "Footprint" "Capacitor_SMD:C_1206_3216Metric" (at 268.9352 213.36 0)
+    (property "Footprint" "Capacitor_SMD:C_0805_2012Metric" (at 268.9352 213.36 0)
       (effects (font (size 1.27 1.27)) hide)
     )

Commit message: Production
Parts:
- C1, C10, C13, C2, C4, C5, C6: LCSC (none) -> C13585
- C11, C12, C3, C7, C8, C9: LCSC (none) -> C913910
- C14: LCSC (none) -> C49217
- D1: LCSC (none) -> C2286
- D2: LCSC (none) -> C2290
- P1: LCSC (none) -> C2927038
- Q1, Q4, Q5, Q8: LCSC (none) -> C15127
- Q2: LCSC (none) -> C908265
- Q3, Q9: LCSC (none) -> C62892
- Q6, Q7: LCSC (none) -> C699266
- R1, R10, R2: LCSC (none) -> C21190
- R11, R12, R13, R14, R21, R25: LCSC (none) -> C25803
- R15, R16, R17, R18, R19, R22, R24, R4, R7, R8: LCSC (none) -> C25804
- R20, R23: LCSC (none) -> C22961
- R3: LCSC (none) -> C22775
- R5, R6: LCSC (none) -> C23179
- U1: LCSC (none) -> C16581
- U2: LCSC (none) -> C917079
- U3: LCSC (none) -> C84681
- U4: LCSC (none) -> C880752
- U5: LCSC (none) -> C89297
- U6: LCSC (none) -> C50506

Commit message: Fabrication
Connections:
- net BTN+: now also D3.6 (K); no longer Q8.1 (G), Q9.6 (C1), R23.2
- net at D3.1 (A): now also Q8.1 (G), Q9.6 (C1), R23.2
Other:
- moved on the sheet: D3A, D3B, D3C, Q8, Q9A, Q9B, R23, R25, SW1, TP11, TP12
