File: PCB/models-heart.kicad_sch (KiCad schematic)
At the start: 103 parts, among them P1 USB_C_Plug, Q1 AO3401A, Q2 FS8205, Q3 UMH3N, Q4 AO3401A, Q5 AO3401A, Q6 BC857BS, Q7 BC857BS, Q8 AO3401A, Q9 UMH3N, SW1 SW_Push, U1 TP4056, U2 DW01, U3 CH340C, U4 AMS1117-3.3, U5 ESP-12E, U6 DRV8833PWP

Commit message: Rev 1
Parts:
- added C15: 0.1uF, Capacitor_SMD:C_0603_1608Metric, symbol Library:C
- added R26, R27: 5k1, Resistor_SMD:R_0603_1608Metric, symbol Library:R
- added R28: 10k, Resistor_SMD:R_0603_1608Metric, symbol Library:R
Connections:
- net +3V3: now also R28.2
- net +PWR SENSE: now also R28.1
- net GND: now also C15.2, R26.2, R27.2
- net at P1.A5 (CC): now also R27.1
- net at P1.B5 (VCONN): now also R26.1
- net at U3.4 (V3): now also C15.1
- no-connect marks 26 -> 23
Other:
- note added: "REV2 * CH340 - Add 0.1uF capasitor to V3 pin * USB Type-C - Add 5k1 resistors to CC pins * ESP8266 - Add Pullup 10k resistor to +PWR Sense line"
- moved on the sheet: C3, C4, Q1, R21, TP10, TP28, TP29, TP42, TP43, TP9

Commit message: actionns test
Connections:
- net USB D+: now also P1.B6 (D+)
- net USB D-: now also P1.B7 (D-)
Changed lines of the file:
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@@
   (junction (at 58.42 97.79) (diameter 0) (color 0 0 0 0)
   )
+  (junction (at 41.91 60.96) (diameter 0) (color 0 0 0 0)
+  )
   (junction (at 294.64 242.57) (diameter 0) (color 0 0 0 0)
   )
@@
   )
   (junction (at 368.3 168.91) (diameter 0) (color 0 0 0 0)
+  )
+  (junction (at 41.91 54.61) (diameter 0) (color 0 0 0 0)
   )
   (junction (at 199.39 130.81) (diameter 0) (color 0 0 0 0)
@@
     (stroke (width 0) (type default))
   )
+  (wire (pts (xy 39.37 57.15) (xy 41.91 57.15))
+    (stroke (width 0) (type default))
+  )
   (wire (pts (xy 142.24 242.57) (xy 144.78 242.57))
     (stroke (width 0) (type default))
@@
   )
   (wire (pts (xy 194.31 130.81) (xy 199.39 130.81))
+    (stroke (width 0) (type default))
+  )
+  (wire (pts (xy 41.91 60.96) (xy 39.37 60.96))
     (stroke (width 0) (type default))
   )
@@
     (stroke (width 0) (type default))
   )
+  (wire (pts (xy 41.91 54.61) (xy 39.37 54.61))
+    (stroke (width 0) (type default))
+  )
   (wire (pts (xy 114.3 124.46) (xy 114.3 129.54))
     (stroke (width 0) (type default))
@@
     (stroke (width 0) (type default))
   )
+  (wire (pts (xy 41.91 57.15) (xy 41.91 54.61))
+    (stroke (width 0) (type default))
+  )
   (wire (pts (xy 354.33 138.43) (xy 354.33 142.24))
     (stroke (width 0) (type default))
@@
     (stroke (width 0) (type default))
   )
+  (wire (pts (xy 41.91 60.96) (xy 48.26 60.96))
+    (stroke (width 0) (type default))
+  )
   (wire (pts (xy 64.77 52.07) (xy 64.77 48.26))
     (stroke (width 0) (type default))
@@
   )
   (wire (pts (xy 106.68 266.7) (xy 106.68 269.24))
-    (stroke (width 0) (type default))
-  )
-  (wire (pts (xy 39.37 55.88) (xy 50.8 55.88))
     (stroke (width 0) (type default))
   )
@@
     (stroke (width 0) (type default))
   )
+  (wire (pts (xy 41.91 63.5) (xy 41.91 60.96))
+    (stroke (width 0) (type default))
+  )
   (wire (pts (xy 259.08 245.11) (xy 260.35 245.11))
     (stroke (width 0) (type default))
@@
     (stroke (width 0) (type default))
   )
-  (wire (pts (xy 39.37 60.96) (xy 53.34 60.96))
-    (stroke (width 0) (type default))
-  )
   (wire (pts (xy 252.73 142.24) (xy 254 142.24))
     (stroke (width 0) (type default))
@@
     (stroke (width 0) (type default))
   )
-  (wire (pts (xy 53.34 60.96) (xy 53.34 77.47))
+  (wire (pts (xy 48.26 60.96) (xy 48.26 77.47))
     (stroke (width 0) (type default))
   )
@@
     (stroke (width 0) (type default))
   )
-  (wire (pts (xy 53.34 77.47) (xy 58.42 77.47))
+  (wire (pts (xy 48.26 77.47) (xy 58.42 77.47))
     (stroke (width 0) (type default))
   )
@@
     (stroke (width 0) (type default))
   )
-  (wire (pts (xy 50.8 55.88) (xy 50.8 80.01))
+  (wire (pts (xy 50.8 54.61) (xy 50.8 80.01))
     (stroke (width 0) (type default))
   )
@@
   )
   (wire (pts (xy 151.13 250.19) (xy 151.13 245.11))
+    (stroke (width 0) (type default))
+  )
+  (wire (pts (xy 41.91 54.61) (xy 50.8 54.61))
     (stroke (width 0) (type default))
   )
@@
     (stroke (width 0) (type default))
   )
+  (wire (pts (xy 39.37 63.5) (xy 41.91 63.5))
+    (stroke (width 0) (type default))
+  )
   (wire (pts (xy 242.57 78.74) (xy 242.57 82.55))
     (stroke (width 0) (type default))
@@
     (effects (font (size 1.27 1.27)) (justify left bottom))
   )
-  (label "USB D+" (at 39.37 60.96 0) (fields_autoplaced)
-    (effects (font (size 1.27 1.27)) (justify left bottom))
-  )
-  (label "USB D-" (at 39.37 55.88 0) (fields_autoplaced)
+  (label "USB D+" (at 41.91 60.96 0) (fields_autoplaced)
+    (effects (font (size 1.27 1.27)) (justify left bottom))
+  )
+  (label "USB D-" (at 41.91 54.61 0) (fields_autoplaced)
     (effects (font (size 1.27 1.27)) (justify left bottom))
   )
@@
     (pin "A5")
     (pin "A6")
+    (pin "B6")
     (pin "A7")
+    (pin "B7")
     (pin "A8")
     (pin "A9")

Commit message: power cutoff
Parts:
- R16: value 10k -> 100k; LCSC C25804 -> C25803
Other:
- note added: "REV2 * CH340 - Add 0.1uF capasitor to V3 pin * USB Type-C - Add 5k1 resistors to CC pins * ESP8266 - Add Pullup 10k resistor to +PWR Sense line * R16 - Change from 10k to 100k - to measure correct battary volrage values"
- note removed: "REV2 * CH340 - Add 0.1uF capasitor to V3 pin * USB Type-C - Add 5k1 resistors to CC pins * ESP8266 - Add Pullup 10k resistor to +PWR Sense line"
Changed lines of the file:
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@@
     (stroke (width 0) (type default))
   )
-  (wire (pts (xy 200.66 224.79) (xy 203.2 224.79))
+  (wire (pts (xy 199.39 224.79) (xy 203.2 224.79))
     (stroke (width 0) (type default))
   )
@@
     (effects (font (size 1.27 1.27)) (justify left bottom))
   )
-  (text "REV2\n* CH340 - Add 0.1uF capasitor to V3 pin\n* USB Type-C - Add 5k1 resistors to CC pins\n* ESP8266 - Add Pullup 10k resistor to +PWR Sense line"
+  (text "REV2\n* CH340 - Add 0.1uF capasitor to V3 pin\n* USB Type-C - Add 5k1 resistors to CC pins\n* ESP8266 - Add Pullup 10k resistor to +PWR Sense line\n* R16 - Change from 10k to 100k - to measure correct battary volrage values"
     (at 15.24 281.94 0)
     (effects (font (size 1.27 1.27)) (justify left bottom))
@@
     )
   )
-  (global_label "A1" (shape input) (at 200.66 224.79 180) (fields_autoplaced)
+  (global_label "A1" (shape input) (at 199.39 224.79 180) (fields_autoplaced)
     (effects (font (size 1.27 1.27)) (justify right))
-    (property "Intersheetrefs" "${INTERSHEET_REFS}" (at 195.4561 224.79 0)
+    (property "Intersheetrefs" "${INTERSHEET_REFS}" (at 194.1861 224.79 0)
       (effects (font (size 1.27 1.27)) (justify right) hide)
     )
@@
     (pin "A5")
     (pin "A6")
-    (pin "B6")
     (pin "A7")
-    (pin "B7")
     (pin "A8")
     (pin "A9")
@@
     (pin "B4")
     (pin "B5")
+    (pin "B6")
+    (pin "B7")
     (pin "B8")
     (pin "B9")
@@
       (effects (font (size 1.27 1.27)))
     )
-    (property "Value" "10k" (at 196.85 201.93 90)
+    (property "Value" "100k" (at 196.85 201.93 90)
       (effects (font (size 1.27 1.27)))
     )
@@
       (effects (font (size 1.27 1.27)) hide)
     )
-    (property "LCSC" "C25804" (at 196.85 205.74 0)
+    (property "LCSC" "C25803" (at 196.85 205.74 0)
       (effects (font (size 1.27 1.27)) hide)
     )

Commit message: REV2
Parts:
- removed P1: USB_C_Plug, Connector_USB:USB_C_Receptacle_GCT_USB4105-xx-A_16P_TopMnt_Horizontal, symbol Library:USB_C_Plug
- removed TP12: BTN, TestPoint:TestPoint_Pad_D1.0mm, symbol Connector:TestPoint_Small
- removed TP28, TP29, TP9: +5V0, TestPoint:TestPoint_Pad_D1.0mm, symbol Connector:TestPoint_Small
- removed TP30, TP32: RX, TestPoint:TestPoint_Pad_D1.0mm, symbol Connector:TestPoint_Small
- removed TP31, TP33: TX, TestPoint:TestPoint_Pad_D1.0mm, symbol Connector:TestPoint_Small
- removed TP34, TP35: RST, TestPoint:TestPoint_Pad_D1.0mm, symbol Connector:TestPoint_Small
- removed TP36, TP37: IO 0, TestPoint:TestPoint_Pad_D1.0mm, symbol Connector:TestPoint_Small
- removed TP38, TP39: D-, TestPoint:TestPoint_Pad_D1.0mm, symbol Connector:TestPoint_Small
- removed TP40, TP41: D+, TestPoint:TestPoint_Pad_D1.0mm, symbol Connector:TestPoint_Small
- removed TP42, TP43, TP7: GND, TestPoint:TestPoint_Pad_D1.0mm, symbol Connector:TestPoint_Small
- removed TP5: BAT -, TestPoint:TestPoint_Pad_D1.0mm, symbol Connector:TestPoint_Small
- removed TP6: BAT +, TestPoint:TestPoint_Pad_D1.0mm, symbol Connector:TestPoint_Small
- added C16, C17: 0.1uF, Capacitor_SMD:C_0603_1608Metric, symbol Library:C
- added J1: USB_C_Receptacle, Connector_USB:USB_C_Receptacle_GCT_USB4115-03-C, symbol Library:USB_C_Receptacle
- added R29: 15k, Resistor_SMD:R_0603_1608Metric, symbol Library:R
- added R30: 100k, Resistor_SMD:R_0603_1608Metric, symbol Library:R
- added TP5: GND, TestPoint:TestPoint_Pad_D1.0mm, symbol Library:TestPoint_Small
- added TP6: NTC, TestPoint:TestPoint_Pad_D1.0mm, symbol Library:TestPoint_Small
- added U7: TPS3808DBV, Package_TO_SOT_SMD:SOT-23-6, symbol Library:TPS3808DBV
- C2: value 10uF -> 0.1uF; footprint Capacitor_SMD:C_1206_3216Metric -> Capacitor_SMD:C_0603_1608Metric; LCSC C13585 -> C913910
- TP1, TP10, TP11, TP13, TP14, TP15, TP16, TP17, TP18, TP19, TP2, TP20, TP21, TP22, TP23, TP24, TP25, TP26, TP27, TP3, TP4, TP8: symbol Connector:TestPoint_Small -> Library:TestPoint_Small
Connections:
- net +3V3: now also R18.2, C16.1, R30.2, U7.6 (VDD); no longer R18.1
- net +5V0 USB: now also J1.A4 (VBUS), J1.A9 (VBUS), J1.B4 (VBUS), J1.B9 (VBUS)
- net BAT +: now also C2.1; no longer C2.2
- net ESP RST: now also U7.1 (~{RESET})
- net GND: now also C2.2, C16.2, C17.2, J1.A1 (GND), J1.A12 (GND), J1.B1 (GND), J1.B12 (GND), J1.S1 (SHIELD), R29.2, TP5.1, U7.2 (GND); no longer C2.1
- net USB D+: now also J1.A6 (D+), J1.B6 (D+)
- net USB D-: now also J1.A7 (D-), J1.B7 (D-)
- net at R27.1: now also J1.A5 (CC1)
- net at R26.1: now also J1.B5 (CC2)
- net at R4.2, R7.1, R9.1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: now also TP6.1
- net at U5.3 (EN): now also R18.1; no longer R18.2
- new net: C17.1, R29.1, R30.1, U7.5 (SENSE)
- no-connect marks 23 -> 25
Other:
- note added: "PWR ADC 4.2V 1V 3,3V 0,7858V"
- note added: "REV2 * CH340 - Add 0.1uF capasitor to V3 pin * USB Type-C - Add 5k1 resistors to CC pins * ESP8266 - Add Pullup 10k resistor to +PWR Sense line * R16 - Change from 10k to 100k - to measure correct battary volrage values * NTC Add termal pin to battary connector"
- note added: "SENSE 0.4V"
- note removed: "REV2 * CH340 - Add 0.1uF capasitor to V3 pin * USB Type-C - Add 5k1 resistors to CC pins * ESP8266 - Add Pullup 10k resistor to +PWR Sense line * R16 - Change from 10k to 100k - to measure correct battary volrage values"
- moved on the sheet: BT1, C10, C11, C5, C6, C7, C8, C9, D3A, D3B, D3C, Q8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

Commit message: placement
Parts:
- removed TP26, TP27: PWR, TestPoint:TestPoint_Pad_D1.0mm, symbol Library:TestPoint_Small
- added H1, H2: MountingHole, MountingHole:MountingHole_2.2mm_M2, symbol Mechanical:MountingHole
- added H3, H4: MountingHole_Pad, MountingHole:MountingHole_2.2mm_M2_Pad_Via, symbol Mechanical:MountingHole_Pad
- added TP12, TP28, TP29, TP7: GND, TestPoint:TestPoint_Pad_D1.0mm, symbol Library:TestPoint_Small
- added TP9: PWR, TestPoint:TestPoint_Pad_D1.0mm, symbol Library:TestPoint_Small
- C11, C12, C15, C16, C17, C3, C7, C8, C9: value 0.1uF -> 100n; footprint Capacitor_SMD:C_0603_1608Metric -> Capacitor_SMD:C_0402_1005Metric; LCSC C913910 -> C307331
- C2: value 0.1uF -> 10uF; footprint Capacitor_SMD:C_0603_1608Metric -> Capacitor_SMD:C_1206_3216Metric; LCSC C913910 -> C13585
- R1, R10, R11, R12, R13, R14, R15, R16, R17, R18, R19, R2, R20, R21, R22, R23, R24, R25, R26, R27, R28, R29, R3, R30, R4, R5, R6, R7, R8: footprint Resistor_SMD:R_0603_1608Metric -> Resistor_SMD:R_0402_1005Metric
- SW1: footprint Button_Switch_SMD:SW_SPST_EVQP7C -> Button_Switch_SMD:SW_Push_SPST_NO_Alps_SKRK; LCSC C115362 -> C2905174
Connections:
- net +PWR: now also TP9.1
- net BAT +: now also C2.2; no longer C2.1
- net GND: now also C2.1, H3.1, H4.1, TP12.1, TP28.1, TP29.1, TP7.1; no longer C2.2
Other:
- moved on the sheet: TP18, TP19, TP20, TP21, TP22, TP23, TP24, TP25
